File: DIYGeiger/DIYGeiger.brd (EAGLE design)
At the start: 144 x 50.2 mm, 0 parts

Commit message: Update
Other:
- board size 144 x 50.2 mm -> 150 x 85 mm
Changed lines of the file:
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@@
 <hole x="-51" y="-6.2" drill="3"/>
 <hole x="-23.5" y="-6.2" drill="3"/>
+<hole x="4.5" y="-16.2" drill="3"/>
+<hole x="4.5" y="-27.2" drill="3"/>
+<hole x="74.5" y="-16.2" drill="3"/>
+<hole x="74.5" y="-27.2" drill="3"/>
+<wire x1="-19" y1="-18" x2="-19" y2="-26" width="0.1524" layer="20"/>
+<wire x1="-19" y1="-26" x2="93" y2="-26" width="0.1524" layer="20"/>
+<wire x1="93" y1="-26" x2="93" y2="-18" width="0.1524" layer="20"/>
+<wire x1="93" y1="-18" x2="-19" y2="-18" width="0.1524" layer="20"/>
+<wire x1="-55" y1="50" x2="-55" y2="-35" width="0.1524" layer="20"/>
+<wire x1="-55" y1="-35" x2="95" y2="-35" width="0.1524" layer="20"/>
+<wire x1="95" y1="-35" x2="95" y2="50" width="0.1524" layer="20"/>
+<wire x1="95" y1="50" x2="-55" y2="50" width="0.1524" layer="20"/>
 </plain>
 <attributes>
